Commit message: replaced dae with stl for UR10

File: Universal_Robots/ur10/urdf/ur10.urdf (robot description, URDF)
Before this commit: robot ur10, 9 links, 8 joints
Links:
- link base_link: geometry collision mesh filename=../meshes/collision/Base.stl; visual mesh filename=../meshes/visual/Base.stl
- link forearm_link: geometry collision mesh filename=../meshes/collision/Forearm.stl; visual mesh filename=../meshes/visual/Forearm.stl
- link shoulder_link: geometry collision mesh filename=../meshes/collision/Shoulder.stl; visual mesh filename=../meshes/visual/Shoulder.stl
- link upper_arm_link: geometry collision mesh filename=../meshes/collision/UpperArm.stl; visual mesh filename=../meshes/visual/UpperArm.stl
- link wrist_1_link: geometry collision mesh filename=../meshes/collision/Wrist1.stl; visual mesh filename=../meshes/visual/Wrist1.stl
- link wrist_2_link: geometry collision mesh filename=../meshes/collision/Wrist2.stl; visual mesh filename=../meshes/visual/Wrist2.stl
- link wrist_3_link: geometry collision mesh filename=../meshes/collision/Wrist3.stl; visual mesh filename=../meshes/visual/Wrist3.stl
