Commit message: added Kinova model, modified UR10 model

File: Universal_Robots/ur10/ur10.urdf (robot description, URDF)
Before this commit: robot ur10, 9 links, 8 joints
Links:
- link base_link: geometry collision mesh filename=./meshes/collision/Base.dae; visual mesh filename=./meshes/visual/Base.dae
- link forearm_link: geometry collision mesh filename=./meshes/collision/Forearm.dae; visual mesh filename=./meshes/visual/Forearm.dae
- link shoulder_link: geometry collision mesh filename=./meshes/collision/Shoulder.dae; visual mesh filename=./meshes/visual/Shoulder.dae
- link upper_arm_link: geometry collision mesh filename=./meshes/collision/UpperArm.dae; visual mesh filename=./meshes/visual/UpperArm.dae
- link wrist_1_link: geometry collision mesh filename=./meshes/collision/Wrist1.dae; visual mesh filename=./meshes/visual/Wrist1.dae
- link wrist_2_link: geometry collision mesh filename=./meshes/collision/Wrist2.dae; visual mesh filename=./meshes/visual/Wrist2.dae
- link wrist_3_link: geometry collision mesh filename=./meshes/collision/Wrist3.dae; visual mesh filename=./meshes/visual/Wrist3.dae

Commit message: stl ur10

File: Universal_Robots/ur10/ur10.urdf (robot description, URDF)
Before this commit: robot ur10, 9 links, 8 joints
Links:
- link base_link: geometry collision mesh filename=./meshes/collision/Base.stl; visual mesh filename=./meshes/visual/Base.stl
- link forearm_link: geometry collision mesh filename=./meshes/collision/Forearm.stl; visual mesh filename=./meshes/visual/Forearm.stl
- link shoulder_link: geometry collision mesh filename=./meshes/collision/Shoulder.stl; visual mesh filename=./meshes/visual/Shoulder.stl
- link upper_arm_link: geometry collision mesh filename=./meshes/collision/UpperArm.stl; visual mesh filename=./meshes/visual/UpperArm.stl
- link wrist_1_link: geometry collision mesh filename=./meshes/collision/Wrist1.stl; visual mesh filename=./meshes/visual/Wrist1.stl
- link wrist_2_link: geometry collision mesh filename=./meshes/collision/Wrist2.stl; visual mesh filename=./meshes/visual/Wrist2.stl
- link wrist_3_link: geometry collision mesh filename=./meshes/collision/Wrist3.stl; visual mesh filename=./meshes/visual/Wrist3.stl

Commit message: fixed world_joint to pos 0,0,0

File: Universal_Robots/ur10/ur10.urdf (robot description, URDF)
Before this commit: robot ur10, 9 links, 8 joints
Joints:
- joint world_joint: origin xyz=0.0 0.0 1.0 rpy=0.0 0.0 0.0 -> xyz=0.0 0.0 0.0 rpy=0.0 0.0 0.0
