Commit message: Franka Panda working

File: Franka/Panda/franka.urdf (robot description, URDF)
Before this commit: robot panda, 13 links, 12 joints
Links:
- link panda_hand: geometry collision mesh filename=./meshes/collision/hand.stl; visual mesh filename=./meshes/visual/hand.dae
- link panda_leftfinger: geometry collision mesh filename=./meshes/collision/finger.stl; visual mesh filename=./meshes/visual/finger.dae
- link panda_link0: geometry collision mesh filename=./meshes/collision/link0.stl; visual mesh filename=./meshes/visual/link0.dae
- link panda_link1: geometry collision mesh filename=./meshes/collision/link1.stl; visual mesh filename=./meshes/visual/link1.dae
- link panda_link2: geometry collision mesh filename=./meshes/collision/link2.stl; visual mesh filename=./meshes/visual/link2.dae
- link panda_link3: geometry collision mesh filename=./meshes/collision/link3.stl; visual mesh filename=./meshes/visual/link3.dae
- link panda_link4: geometry collision mesh filename=./meshes/collision/link4.stl; visual mesh filename=./meshes/visual/link4.dae
- link panda_link5: geometry collision mesh filename=./meshes/collision/link5.stl; visual mesh filename=./meshes/visual/link5.dae
- link panda_link6: geometry collision mesh filename=./meshes/collision/link6.stl; visual mesh filename=./meshes/visual/link6.dae
- link panda_link7: geometry collision mesh filename=./meshes/collision/link7.stl; visual mesh filename=./meshes/visual/link7.dae
- link panda_rightfinger: geometry collision mesh filename=./meshes/collision/finger.stl; visual mesh filename=./meshes/visual/finger.dae
