Commit message: minor

File: Universal_Robots/ur10_robotiq_2f_85/ur10_robot.urdf (robot description, URDF)
Before this commit: robot ur10, 22 links, 21 joints
Links:
- link gripper_left_inner_finger: geometry collision mesh filename=./robotiq_2f_85_gripper_visualization/meshes/collision/robo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 scale=0.001 0.001 0.001; visual mesh filename=./robotiq_2f_85_gripper_visualization/meshes/visual/robotiq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 scale=0.001 0.001 0.001
- link gripper_left_inner_knuckle: geometry collision mesh filename=./robotiq_2f_85_gripper_visualization/meshes/collision/robo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 scale=0.001 0.001 0.001; visual mesh filename=./robotiq_2f_85_gripper_visualization/meshes/visual/robotiq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 scale=0.001 0.001 0.001
- link gripper_left_outer_finger: geometry collision mesh filename=./robotiq_2f_85_gripper_visualization/meshes/collision/robo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 scale=0.001 0.001 0.001; visual mesh filename=./robotiq_2f_85_gripper_visualization/meshes/visual/robotiq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 scale=0.001 0.001 0.001
- link gripper_left_outer_knuckle: geometry collision mesh filename=./robotiq_2f_85_gripper_visualization/meshes/collision/robo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 scale=0.001 0.001 0.001; visual mesh filename=./robotiq_2f_85_gripper_visualization/meshes/visual/robotiq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 scale=0.001 0.001 0.001
- link gripper_right_inner_finger: geometry collision mesh filename=./robotiq_2f_85_gripper_visualization/meshes/collision/robo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 scale=0.001 0.001 0.001; visual mesh filename=./robotiq_2f_85_gripper_visualization/meshes/visual/robotiq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 scale=0.001 0.001 0.001
- link gripper_right_inner_knuckle: geometry collision mesh filename=./robotiq_2f_85_gripper_visualization/meshes/collision/robo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 scale=0.001 0.001 0.001; visual mesh filename=./robotiq_2f_85_gripper_visualization/meshes/visual/robotiq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 scale=0.001 0.001 0.001
- link gripper_right_outer_finger: geometry collision mesh filename=./robotiq_2f_85_gripper_visualization/meshes/collision/robo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 scale=0.001 0.001 0.001; visual mesh filename=./robotiq_2f_85_gripper_visualization/meshes/visual/robotiq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 scale=0.001 0.001 0.001
- link gripper_right_outer_knuckle: geometry collision mesh filename=./robotiq_2f_85_gripper_visualization/meshes/collision/robo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 scale=0.001 0.001 0.001; visual mesh filename=./robotiq_2f_85_gripper_visualization/meshes/visual/robotiq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 scale=0.001 0.001 0.001
- link gripper_robotiq_arg2f_base_link: geometry collision mesh filename=./robotiq_2f_85_gripper_visualization/meshes/collision/robo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; visual mesh filename=./robotiq_2f_85_gripper_visualization/meshes/visual/robotiq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 scale=0.001 0.001 0.001
- link robot_base_link: geometry collision mesh filename=./ur_description/meshes/ur10/collision/base.stl; visual mesh filename=./ur_description/meshes/ur10/visual/base.dae
- link robot_forearm_link: geometry collision mesh filename=./ur_description/meshes/ur10/collision/forearm.stl; visual mesh filename=./ur_description/meshes/ur10/visual/forearm.dae
- link robot_shoulder_link: geometry collision mesh filename=./ur_description/meshes/ur10/collision/shoulder.stl; visual mesh filename=./ur_description/meshes/ur10/visual/shoulder.dae
- link robot_upper_arm_link: geometry collision mesh filename=./ur_description/meshes/ur10/collision/upperarm.stl; visual mesh filename=./ur_description/meshes/ur10/visual/upperarm.dae
- link robot_wrist_1_link: geometry collision mesh filename=./ur_description/meshes/ur10/collision/wrist1.stl; visual mesh filename=./ur_description/meshes/ur10/visual/wrist1.dae
- link robot_wrist_2_link: geometry collision mesh filename=./ur_description/meshes/ur10/collision/wrist2.stl; visual mesh filename=./ur_description/meshes/ur10/visual/wrist2.dae
- link robot_wrist_3_link: geometry collision mesh filename=./ur_description/meshes/ur10/collision/wrist3.stl; visual mesh filename=./ur_description/meshes/ur10/visual/wrist3.dae

File: Universal_Robots/ur10_robotiq_2f_85/ur10_robot_constr.urdf (robot description, URDF)
Before this commit: robot ur10, 22 links, 21 joints
Links:
- link gripper_left_inner_finger: geometry collision mesh filename=./robotiq_2f_85_gripper_visualization/meshes/collision/robo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 scale=0.001 0.001 0.001; visual mesh filename=./robotiq_2f_85_gripper_visualization/meshes/visual/robotiq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 scale=0.001 0.001 0.001
- link gripper_left_inner_knuckle: geometry collision mesh filename=./robotiq_2f_85_gripper_visualization/meshes/collision/robo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 scale=0.001 0.001 0.001; visual mesh filename=./robotiq_2f_85_gripper_visualization/meshes/visual/robotiq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 scale=0.001 0.001 0.001
- link gripper_left_outer_finger: geometry collision mesh filename=./robotiq_2f_85_gripper_visualization/meshes/collision/robo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 scale=0.001 0.001 0.001; visual mesh filename=./robotiq_2f_85_gripper_visualization/meshes/visual/robotiq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 scale=0.001 0.001 0.001
- link gripper_left_outer_knuckle: geometry collision mesh filename=./robotiq_2f_85_gripper_visualization/meshes/collision/robo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 scale=0.001 0.001 0.001; visual mesh filename=./robotiq_2f_85_gripper_visualization/meshes/visual/robotiq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 scale=0.001 0.001 0.001
- link gripper_right_inner_finger: geometry collision mesh filename=./robotiq_2f_85_gripper_visualization/meshes/collision/robo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 scale=0.001 0.001 0.001; visual mesh filename=./robotiq_2f_85_gripper_visualization/meshes/visual/robotiq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 scale=0.001 0.001 0.001
- link gripper_right_inner_knuckle: geometry collision mesh filename=./robotiq_2f_85_gripper_visualization/meshes/collision/robo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 scale=0.001 0.001 0.001; visual mesh filename=./robotiq_2f_85_gripper_visualization/meshes/visual/robotiq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 scale=0.001 0.001 0.001
- link gripper_right_outer_finger: geometry collision mesh filename=./robotiq_2f_85_gripper_visualization/meshes/collision/robo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 scale=0.001 0.001 0.001; visual mesh filename=./robotiq_2f_85_gripper_visualization/meshes/visual/robotiq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 scale=0.001 0.001 0.001
- link gripper_right_outer_knuckle: geometry collision mesh filename=./robotiq_2f_85_gripper_visualization/meshes/collision/robo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 scale=0.001 0.001 0.001; visual mesh filename=./robotiq_2f_85_gripper_visualization/meshes/visual/robotiq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 scale=0.001 0.001 0.001
- link gripper_robotiq_arg2f_base_link: geometry collision mesh filename=./robotiq_2f_85_gripper_visualization/meshes/collision/robo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; visual mesh filename=./robotiq_2f_85_gripper_visualization/meshes/visual/robotiq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 scale=0.001 0.001 0.001
- link robot_base_link: geometry collision mesh filename=./ur_description/meshes/ur10/collision/base.stl; visual mesh filename=./ur_description/meshes/ur10/visual/base.dae
- link robot_forearm_link: geometry collision mesh filename=./ur_description/meshes/ur10/collision/forearm.stl; visual mesh filename=./ur_description/meshes/ur10/visual/forearm.dae
- link robot_shoulder_link: geometry collision mesh filename=./ur_description/meshes/ur10/collision/shoulder.stl; visual mesh filename=./ur_description/meshes/ur10/visual/shoulder.dae
- link robot_upper_arm_link: geometry collision mesh filename=./ur_description/meshes/ur10/collision/upperarm.stl; visual mesh filename=./ur_description/meshes/ur10/visual/upperarm.dae
- link robot_wrist_1_link: geometry collision mesh filename=./ur_description/meshes/ur10/collision/wrist1.stl; visual mesh filename=./ur_description/meshes/ur10/visual/wrist1.dae
- link robot_wrist_2_link: geometry collision mesh filename=./ur_description/meshes/ur10/collision/wrist2.stl; visual mesh filename=./ur_description/meshes/ur10/visual/wrist2.dae
- link robot_wrist_3_link: geometry collision mesh filename=./ur_description/meshes/ur10/collision/wrist3.stl; visual mesh filename=./ur_description/meshes/ur10/visual/wrist3.dae
