Commit message: minor

File: Universal_Robots/ur10_robotiq_2f_85/ur10.urdf (robot description, URDF)
Before this commit: robot ur10, 21 links, 20 joints
Links:
- removed link EE_robotiq_2f85
- removed link robotiq_85_base_link
- removed link robotiq_85_left_finger_link
- removed link robotiq_85_left_finger_tip_link
- removed link robotiq_85_left_inner_knuckle_link
- removed link robotiq_85_left_knuckle_link
- removed link robotiq_85_right_finger_link
- removed link robotiq_85_right_finger_tip_link
- removed link robotiq_85_right_inner_knuckle_link
- removed link robotiq_85_right_knuckle_link
- removed link robotiq_coupler
Joints:
- removed joint EE_robotiq_2f85_joint
- removed joint robotiq_85_base_joint
- removed joint robotiq_85_left_finger_joint
- removed joint robotiq_85_left_finger_tip_joint
- removed joint robotiq_85_left_inner_knuckle_joint
- removed joint robotiq_85_left_knuckle_joint
- removed joint robotiq_85_right_finger_joint
- removed joint robotiq_85_right_finger_tip_joint
- removed joint robotiq_85_right_inner_knuckle_joint
- removed joint robotiq_85_right_knuckle_joint
- removed joint robotiq_coupler_joint

Commit message: minor

File: Universal_Robots/ur10_robotiq_2f_85/ur10.urdf (robot description, URDF)
Before this commit: robot ur10, 10 links, 9 joints
Links:
- added link robotiq_coupler, mass 0.168; collision mesh filename=./meshes/robotiq2f85/robotiq_85_coupler.stl; visual mesh filename=./meshes/robotiq2f85/robotiq_85_coupler.stl
Joints:
- added joint robotiq_coupler_joint: type fixed, parent tool0, child robotiq_coupler, origin xyz=0 0 0.004 rpy=0 0 -1.57079632679

Commit message: minor

File: Universal_Robots/ur10_robotiq_2f_85/ur10.urdf (robot description, URDF)
Before this commit: robot ur10, 11 links, 10 joints
Links:
- added link robotiq_85_base_link, mass 0.636951; collision mesh filename=./meshes/robotiq2f85/collision/robotiq_85_base_link.stl; visual mesh filename=./meshes/robotiq2f85/visual/robotiq_85_base_link.dae
Joints:
- added joint robotiq_85_base_joint: type fixed, parent robotiq_coupler, child robotiq_85_base_link, origin xyz=0 0 0.004 rpy=0 -1.57079632679 3.141592653

Commit message: added robotiq_85_left_knuckle_link

File: Universal_Robots/ur10_robotiq_2f_85/ur10.urdf (robot description, URDF)
Before this commit: robot ur10, 12 links, 11 joints
Links:
- added link robotiq_85_left_knuckle_link, mass 0.018491; collision mesh filename=./meshes/robotiq2f85/collision/robotiq_85_knuckle_link.stl; visual mesh filename=./meshes/robotiq2f85/visual/robotiq_85_knuckle_link.dae
Joints:
- added joint robotiq_85_left_knuckle_joint: type revolute, parent robotiq_85_base_link, child robotiq_85_left_knuckle_link, origin xyz=0.05490451627 0.03060114443 0.0 rpy=3.141592653 0.0 0.0, axis 0 0 1, limit lower=-0.05 upper=0.80285 effort=1000 velocity=0.5

Commit message: testing

File: Universal_Robots/ur10_robotiq_2f_85/ur10.urdf (robot description, URDF)
Before this commit: robot ur10, 13 links, 12 joints
Links:
- added link EE_robotiq_2f85, mass 0.00001; visual box size=0.001 0.001 0.001
- added link robotiq_85_left_finger_link, mass 0.027309; collision mesh filename=./meshes/robotiq2f85/collision/robotiq_85_finger_link.stl; visual mesh filename=./meshes/robotiq2f85/visual/robotiq_85_finger_link.dae
- added link robotiq_85_left_finger_tip_link, mass 0.019555; collision mesh filename=./meshes/robotiq2f85/collision/robotiq_85_finger_tip_link.s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; visual mesh filename=./meshes/robotiq2f85/visual/robotiq_85_finger_tip_link.dae
- added link robotiq_85_left_inner_knuckle_link, mass 0.029951; collision mesh filename=./meshes/robotiq2f85/collision/robotiq_85_inner_knuckle_lin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; visual mesh filename=./meshes/robotiq2f85/visual/robotiq_85_inner_knuckle_link.d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
- added link robotiq_85_right_finger_link, mass 0.027309; collision mesh filename=./meshes/robotiq2f85/collision/robotiq_85_finger_link.stl; visual mesh filename=./meshes/robotiq2f85/visual/robotiq_85_finger_link.dae
- added link robotiq_85_right_finger_tip_link, mass 0.019555; collision mesh filename=./meshes/robotiq2f85/collision/robotiq_85_finger_tip_link.s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; visual mesh filename=./meshes/robotiq2f85/visual/robotiq_85_finger_tip_link.dae
- added link robotiq_85_right_inner_knuckle_link, mass 0.029951; collision mesh filename=./meshes/robotiq2f85/collision/robotiq_85_inner_knuckle_lin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; visual mesh filename=./meshes/robotiq2f85/visual/robotiq_85_inner_knuckle_link.d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
- added link robotiq_85_right_knuckle_link, mass 0.018491; collision mesh filename=./meshes/robotiq2f85/collision/robotiq_85_knuckle_link.stl; visual mesh filename=./meshes/robotiq2f85/visual/robotiq_85_knuckle_link.dae
Joints:
- added joint EE_robotiq_2f85_joint: type prismatic, parent robotiq_85_base_link, child EE_robotiq_2f85, origin xyz=0.128 0.0 0.0 rpy=0 0 0, axis 1 0 0, limit lower=0.0 upper=0.0 effort=10000 velocity=0.0
- added joint robotiq_85_left_finger_joint: type fixed, parent robotiq_85_left_knuckle_link, child robotiq_85_left_finger_link, origin xyz=-0.00408552455 -0.03148604435 0.0 rpy=0 0 0
- added joint robotiq_85_left_finger_tip_joint: type continuous, parent robotiq_85_left_inner_knuckle_link, child robotiq_85_left_finger_tip_link, origin xyz=0.04303959807 -0.03759940821 0.0 rpy=0.0 0.0 0.0, axis 0 0 1, limit lower=-0.80285 upper=0.05 effort=1000 velocity=0.5
- added joint robotiq_85_left_inner_knuckle_joint: type continuous, parent robotiq_85_base_link, child robotiq_85_left_inner_knuckle_link, origin xyz=0.06142 0.0127 0 rpy=${pi} 0.0 0.0, axis 0 0 1, limit lower=-0.05 upper=0.80285 effort=1000 velocity=0.5
- added joint robotiq_85_right_finger_joint: type fixed, parent robotiq_85_right_knuckle_link, child robotiq_85_right_finger_link, origin xyz=-0.00408552455 -0.03148604435 0.0 rpy=0 0 0
- added joint robotiq_85_right_finger_tip_joint: type continuous, parent robotiq_85_right_inner_knuckle_link, child robotiq_85_right_finger_tip_link, origin xyz=0.04303959807 -0.03759940821  0.0 rpy=0.0 0.0 0.0, axis 0 0 1, limit lower=-0.80285 upper=0.05 effort=1000 velocity=0.5
- added joint robotiq_85_right_inner_knuckle_joint: type continuous, parent robotiq_85_base_link, child robotiq_85_right_inner_knuckle_link, origin xyz=0.06142 -0.0127 0 rpy=0 0 0, axis 0 0 1, limit lower=-0.05 upper=0.80285 effort=1000 velocity=0.5
- added joint robotiq_85_right_knuckle_joint: type continuous, parent robotiq_85_base_link, child robotiq_85_right_knuckle_link, origin xyz=0.05490451627 -0.03060114443 0.0 rpy=0.0 0.0 0.0, axis 0 0 1, limit lower=-0.05 upper=0.80285 effort=1000 velocity=0.5

Commit message: minor

File: Universal_Robots/ur10_robotiq_2f_85/ur10.urdf (robot description, URDF)
Before this commit: robot ur10, 12 links, 11 joints
Links:
- removed link robotiq_85_base_link
Joints:
- removed joint robotiq_85_base_joint

Commit message: test

File: Universal_Robots/ur10_robotiq_2f_85/ur10.urdf (robot description, URDF)
Before this commit: robot ur10, 11 links, 10 joints
Links:
- added link EE_robotiq_2f85, mass 0.00001; visual box size=0.001 0.001 0.001
- added link robotiq_85_base_link, mass 0.636951; collision mesh filename=./meshes/robotiq2f85/collision/robotiq_85_base_link.stl; visual mesh filename=./meshes/robotiq2f85/visual/robotiq_85_base_link.dae
- added link robotiq_85_left_finger_link, mass 0.027309; collision mesh filename=./meshes/robotiq2f85/collision/robotiq_85_finger_link.stl; visual mesh filename=./meshes/robotiq2f85/visual/robotiq_85_finger_link.dae
- added link robotiq_85_left_finger_tip_link, mass 0.019555; collision mesh filename=./meshes/robotiq2f85/collision/robotiq_85_finger_tip_link.s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; visual mesh filename=./meshes/robotiq2f85/visual/robotiq_85_finger_tip_link.dae
- added link robotiq_85_left_inner_knuckle_link, mass 0.029951; collision mesh filename=./meshes/robotiq2f85/collision/robotiq_85_inner_knuckle_lin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; visual mesh filename=./meshes/robotiq2f85/visual/robotiq_85_inner_knuckle_link.d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
- added link robotiq_85_left_knuckle_link, mass 0.018491; collision mesh filename=./meshes/robotiq2f85/collision/robotiq_85_knuckle_link.stl; visual mesh filename=./meshes/robotiq2f85/visual/robotiq_85_knuckle_link.dae
- added link robotiq_85_right_finger_link, mass 0.027309; collision mesh filename=./meshes/robotiq2f85/collision/robotiq_85_finger_link.stl; visual mesh filename=./meshes/robotiq2f85/visual/robotiq_85_finger_link.dae
- added link robotiq_85_right_finger_tip_link, mass 0.019555; collision mesh filename=./meshes/robotiq2f85/collision/robotiq_85_finger_tip_link.s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; visual mesh filename=./meshes/robotiq2f85/visual/robotiq_85_finger_tip_link.dae
- added link robotiq_85_right_inner_knuckle_link, mass 0.029951; collision mesh filename=./meshes/robotiq2f85/collision/robotiq_85_inner_knuckle_lin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; visual mesh filename=./meshes/robotiq2f85/visual/robotiq_85_inner_knuckle_link.d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
- added link robotiq_85_right_knuckle_link, mass 0.018491; collision mesh filename=./meshes/robotiq2f85/collision/robotiq_85_knuckle_link.stl; visual mesh filename=./meshes/robotiq2f85/visual/robotiq_85_knuckle_link.dae
Joints:
- added joint EE_robotiq_2f85_joint: type prismatic, parent robotiq_85_base_link, child EE_robotiq_2f85, origin xyz=0.128 0.0 0.0 rpy=0 0 0, axis 1 0 0, limit lower=0.0 upper=0.0 effort=10000 velocity=0.0
- added joint robotiq_85_base_joint: type fixed, parent robotiq_coupler, child robotiq_85_base_link, origin xyz=0 0 0.004 rpy=0 -1.57079632679 3.141592653
- added joint robotiq_85_left_finger_joint: type fixed, parent robotiq_85_left_knuckle_link, child robotiq_85_left_finger_link, origin xyz=-0.00408552455 -0.03148604435 0.0 rpy=0 0 0
- added joint robotiq_85_left_finger_tip_joint: type continuous, parent robotiq_85_left_inner_knuckle_link, child robotiq_85_left_finger_tip_link, origin xyz=0.04303959807 -0.03759940821 0.0 rpy=0.0 0.0 0.0, axis 0 0 1, limit lower=-0.80285 upper=0.05 effort=1000 velocity=0.5
- added joint robotiq_85_left_inner_knuckle_joint: type continuous, parent robotiq_85_base_link, child robotiq_85_left_inner_knuckle_link, origin xyz=0.06142 0.0127 0 rpy=${pi} 0.0 0.0, axis 0 0 1, limit lower=-0.05 upper=0.80285 effort=1000 velocity=0.5
- added joint robotiq_85_left_knuckle_joint: type revolute, parent robotiq_85_base_link, child robotiq_85_left_knuckle_link, origin xyz=0.05490451627 0.03060114443 0.0 rpy=3.141592653 0.0 0.0, axis 0 0 1, limit lower=-0.05 upper=0.80285 effort=1000 velocity=0.5
- added joint robotiq_85_right_finger_joint: type fixed, parent robotiq_85_right_knuckle_link, child robotiq_85_right_finger_link, origin xyz=-0.00408552455 -0.03148604435 0.0 rpy=0 0 0
- added joint robotiq_85_right_finger_tip_joint: type continuous, parent robotiq_85_right_inner_knuckle_link, child robotiq_85_right_finger_tip_link, origin xyz=0.04303959807 -0.03759940821  0.0 rpy=0.0 0.0 0.0, axis 0 0 1, limit lower=-0.80285 upper=0.05 effort=1000 velocity=0.5
- added joint robotiq_85_right_inner_knuckle_joint: type continuous, parent robotiq_85_base_link, child robotiq_85_right_inner_knuckle_link, origin xyz=0.06142 -0.0127 0 rpy=0 0 0, axis 0 0 1, limit lower=-0.05 upper=0.80285 effort=1000 velocity=0.5
- added joint robotiq_85_right_knuckle_joint: type continuous, parent robotiq_85_base_link, child robotiq_85_right_knuckle_link, origin xyz=0.05490451627 -0.03060114443 0.0 rpy=0.0 0.0 0.0, axis 0 0 1, limit lower=-0.05 upper=0.80285 effort=1000 velocity=0.5

Commit message: minor

File: Universal_Robots/ur10_robotiq_2f_85/ur10.urdf (robot description, URDF)
Before this commit: robot ur10, 21 links, 20 joints
Links:
- removed link ee_link
Joints:
- removed joint ee_fixed_joint
