Commit message: minor

File: Universal_Robots/ur10_robotiq_2f_85/ur10_gripper_b.urdf (robot description, URDF)
Before this commit: robot ur10, 22 links, 21 joints
Links:
- removed link robotiq_85_left_finger_link
- removed link robotiq_85_left_finger_tip_link
- removed link robotiq_85_left_inner_knuckle_link
- removed link robotiq_85_left_knuckle_link
- removed link robotiq_85_right_finger_link
- removed link robotiq_85_right_finger_tip_link
- removed link robotiq_85_right_inner_knuckle_link
- removed link robotiq_85_right_knuckle_link
- added link left_inner_finger, mass 0.00724255346165745; collision mesh filename=./meshes/robotiq2f85/inner_finger_coarse.STL; visual mesh filename=./meshes/robotiq2f85/inner_finger_fine.STL
- added link left_inner_knuckle, mass 0.0110930853895903; collision mesh filename=./meshes/robotiq2f85/inner_knuckle_coarse.STL; visual mesh filename=./meshes/robotiq2f85/inner_knuckle_fine.STL
- added link left_outer_finger, mass 0.0273093985570947; collision mesh filename=./meshes/robotiq2f85/outer_finger_coarse.STL; visual mesh filename=./meshes/robotiq2f85/outer_finger_fine.STL
- added link left_outer_knuckle, mass 0.00684838849434396; collision mesh filename=./meshes/robotiq2f85/outer_knuckle_coarse.STL; visual mesh filename=./meshes/robotiq2f85/outer_knuckle_fine.STL
- added link right_inner_finger, mass 0.00724255346165744; collision mesh filename=./meshes/robotiq2f85/inner_finger_coarse.STL; visual mesh filename=./meshes/robotiq2f85/inner_finger_fine.STL
- added link right_inner_knuckle, mass 0.0110930853895903; collision mesh filename=./meshes/robotiq2f85/inner_knuckle_coarse.STL; visual mesh filename=./meshes/robotiq2f85/inner_knuckle_fine.STL
- added link right_outer_finger, mass 0.0273093985570947; collision mesh filename=./meshes/robotiq2f85/outer_finger_coarse.STL; visual mesh filename=./meshes/robotiq2f85/outer_finger_fine.STL
- added link right_outer_knuckle, mass 0.00684838849401352; collision mesh filename=./meshes/robotiq2f85/outer_knuckle_coarse.STL; visual mesh filename=./meshes/robotiq2f85/outer_knuckle_fine.STL
- link robotiq_85_base_link: mass 0.636951 -> 0.30915
Joints:
- removed joint robotiq_85_left_finger_joint
- removed joint robotiq_85_left_finger_tip_joint
- removed joint robotiq_85_left_inner_knuckle_joint
- removed joint robotiq_85_left_knuckle_joint
- removed joint robotiq_85_right_finger_joint
- removed joint robotiq_85_right_finger_tip_joint
- removed joint robotiq_85_right_inner_knuckle_joint
- removed joint robotiq_85_right_knuckle_joint
- added joint finger_joint: type revolute, parent robotiq_85_base_link, child left_outer_knuckle, origin xyz=0.0306011444260539 0 0.0627920162695395 rpy=0 0 0, axis 0 -1 0, limit lower=0 upper=0.725 effort=1000 velocity=2.0
- added joint left_inner_finger_joint: type revolute, parent left_inner_knuckle, child left_inner_finger, origin xyz=0.034585310861294 0 0.0454970193817975 rpy=0 0 0, axis 0 -1 0, limit lower=0 upper=0.8757 effort=1000 velocity=2.0, mimic joint=finger_joint multiplier=-1 offset=0
- added joint left_inner_knuckle_joint: type revolute, parent robotiq_85_base_link, child left_inner_knuckle, origin xyz=0.0127000000001501 0 0.0693074999999639 rpy=0 0 0, axis 0 -1 0, limit lower=0 upper=0.8757 effort=1000 velocity=2.0, mimic joint=finger_joint multiplier=1 offset=0
- added joint left_outer_finger_joint: type fixed, parent left_outer_knuckle, child left_outer_finger, origin xyz=0.0316910442266543 0 -0.00193396375724605 rpy=0 0 0, axis 0 -1 0
- added joint right_inner_finger_joint: type revolute, parent right_inner_knuckle, child right_inner_finger, origin xyz=0.0341060475457406 0 0.0458573878541688 rpy=0 0 0, axis 0 1 0, limit lower=0 upper=0.8757 effort=1000 velocity=2.0, mimic joint=finger_joint multiplier=1 offset=0
- added joint right_inner_knuckle_joint: type revolute, parent robotiq_85_base_link, child right_inner_knuckle, origin xyz=-0.0126999999998499 0 0.0693075000000361 rpy=0 0 3.14159265358979, axis 0 1 0, limit lower=0 upper=0.8757 effort=1000 velocity=2.0, mimic joint=finger_joint multiplier=-1 offset=0
- added joint right_outer_finger_joint: type fixed, parent right_outer_knuckle, child right_outer_finger, origin xyz=0.0317095909367246 0 -0.0016013564954687 rpy=0 0 0, axis 0 1 0
- added joint right_outer_knuckle_joint: type revolute, parent robotiq_85_base_link, child right_outer_knuckle, origin xyz=-0.0306011444258893 0 0.0627920162695395 rpy=0 0 3.14159265358979, axis 0 1 0, limit lower=0 upper=0.8757 effort=1000 velocity=2.0, mimic joint=finger_joint multiplier=-1 offset=0
- joint robotiq_85_base_joint: origin xyz=0 0 0.004 rpy=0 -1.57079632679 3.141592653 -> xyz=0.5 0 0.004 rpy=0 -1.57079632679 3.141592653
