Commit message: minor

File: Universal_Robots/ur10_robotiq_2f_85/ur10_gripper.urdf (robot description, URDF)
Before this commit: robot ur10, 22 links, 21 joints
Links:
- link base_link: geometry collision mesh filename=./meshes/collision/Base.dae; visual mesh filename=./meshes/visual/Base.dae
- link forearm_link: geometry collision mesh filename=./meshes/collision/Forearm.dae; visual mesh filename=./meshes/visual/Forearm.dae
- link shoulder_link: geometry collision mesh filename=./meshes/collision/Shoulder.dae; visual mesh filename=./meshes/visual/Shoulder.dae
- link upper_arm_link: geometry collision mesh filename=./meshes/collision/UpperArm.dae; visual mesh filename=./meshes/visual/UpperArm.dae
- link wrist_1_link: geometry collision mesh filename=./meshes/collision/Wrist3.dae; visual mesh filename=./meshes/visual/Wrist3.dae

Commit message: minor

File: Universal_Robots/ur10_robotiq_2f_85/ur10_gripper.urdf (robot description, URDF)
Before this commit: robot ur10, 22 links, 21 joints
Joints:
- joint robot_tool0_gripper_robotiq_arg2f_base_link: origin xyz=0 0 0 rpy=1.57079632679 -1.57079632679 0 -> xyz=0 0 0.004 rpy=0 0 -1.57079632679

Commit message: changed gripper meshes

File: Universal_Robots/ur10_robotiq_2f_85/ur10_gripper.urdf (robot description, URDF)
Before this commit: robot ur10, 22 links, 21 joints
Links:
- removed link gripper_left_inner_finger
- removed link gripper_left_inner_finger_pad
- removed link gripper_left_inner_knuckle
- removed link gripper_left_outer_finger
- removed link gripper_left_outer_knuckle
- removed link gripper_right_inner_finger
- removed link gripper_right_inner_finger_pad
- removed link gripper_right_inner_knuckle
- removed link gripper_right_outer_finger
- removed link gripper_right_outer_knuckle
- removed link gripper_robotiq_arg2f_base_link
- added link EE_robotiq_2f85, mass 0.00001; visual box size=0.001 0.001 0.001
- added link robotiq_85_base_link, mass 0.636951; collision mesh filename=./meshes/robotiq2f85/collision/robotiq_85_base_link.stl; visual mesh filename=./meshes/robotiq2f85/visual/robotiq_85_base_link.dae
- added link robotiq_85_left_finger_link, mass 0.027309; collision mesh filename=./meshes/robotiq2f85/collision/robotiq_85_finger_link.stl; visual mesh filename=./meshes/robotiq2f85/visual/robotiq_85_finger_link.dae
- added link robotiq_85_left_finger_tip_link, mass 0.019555; collision mesh filename=./meshes/robotiq2f85/collision/robotiq_85_finger_tip_link.s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; visual mesh filename=./meshes/robotiq2f85/visual/robotiq_85_finger_tip_link.dae
- added link robotiq_85_left_inner_knuckle_link, mass 0.029951; collision mesh filename=./meshes/robotiq2f85/collision/robotiq_85_inner_knuckle_lin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; visual mesh filename=./meshes/robotiq2f85/visual/robotiq_85_inner_knuckle_link.d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
- added link robotiq_85_left_knuckle_link, mass 0.018491; collision mesh filename=./meshes/robotiq2f85/collision/robotiq_85_knuckle_link.stl; visual mesh filename=./meshes/robotiq2f85/visual/robotiq_85_knuckle_link.dae
- added link robotiq_85_right_finger_link, mass 0.027309; collision mesh filename=./meshes/robotiq2f85/collision/robotiq_85_finger_link.stl; visual mesh filename=./meshes/robotiq2f85/visual/robotiq_85_finger_link.dae
- added link robotiq_85_right_finger_tip_link, mass 0.019555; collision mesh filename=./meshes/robotiq2f85/collision/robotiq_85_finger_tip_link.s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; visual mesh filename=./meshes/robotiq2f85/visual/robotiq_85_finger_tip_link.dae
- added link robotiq_85_right_inner_knuckle_link, mass 0.029951; collision mesh filename=./meshes/robotiq2f85/collision/robotiq_85_inner_knuckle_lin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; visual mesh filename=./meshes/robotiq2f85/visual/robotiq_85_inner_knuckle_link.d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
- added link robotiq_85_right_knuckle_link, mass 0.018491; collision mesh filename=./meshes/robotiq2f85/collision/robotiq_85_knuckle_link.stl; visual mesh filename=./meshes/robotiq2f85/visual/robotiq_85_knuckle_link.dae
- added link robotiq_coupler, mass 0.168; collision mesh filename=./meshes/robotiq2f85/robotiq_85_coupler.stl; visual mesh filename=./meshes/robotiq2f85/robotiq_85_coupler.stl
Joints:
- removed joint gripper_finger_joint
- removed joint gripper_left_inner_finger_joint
- removed joint gripper_left_inner_finger_pad_joint
- removed joint gripper_left_inner_knuckle_joint
- removed joint gripper_left_outer_finger_joint
- removed joint gripper_right_inner_finger_joint
- removed joint gripper_right_inner_finger_pad_joint
- removed joint gripper_right_inner_knuckle_joint
- removed joint gripper_right_outer_finger_joint
- removed joint gripper_right_outer_knuckle_joint
- removed joint robot_tool0_gripper_robotiq_arg2f_base_link
- added joint EE_robotiq_2f85_joint: type prismatic, parent robotiq_85_base_link, child EE_robotiq_2f85, origin xyz=0.128 0.0 0.0 rpy=0 0 0, axis 1 0 0, limit lower=0.0 upper=0.0 effort=10000 velocity=0.0
- added joint robotiq_85_base_joint: type fixed, parent robotiq_coupler, child robotiq_85_base_link, origin xyz=0 0 0.004 rpy=0 -1.57079632679 3.141592653
- added joint robotiq_85_left_finger_joint: type fixed, parent robotiq_85_left_knuckle_link, child robotiq_85_left_finger_link, origin xyz=-0.00408552455 -0.03148604435 0.0 rpy=0 0 0
- added joint robotiq_85_left_finger_tip_joint: type continuous, parent robotiq_85_left_inner_knuckle_link, child robotiq_85_left_finger_tip_link, origin xyz=0.04303959807 -0.03759940821 0.0 rpy=0.0 0.0 0.0, axis 0 0 1, limit lower=-0.80285 upper=0.05 effort=1000 velocity=0.5
- added joint robotiq_85_left_inner_knuckle_joint: type continuous, parent robotiq_85_base_link, child robotiq_85_left_inner_knuckle_link, origin xyz=0.06142 0.0127 0 rpy=${pi} 0.0 0.0, axis 0 0 1, limit lower=-0.05 upper=0.80285 effort=1000 velocity=0.5
- added joint robotiq_85_left_knuckle_joint: type revolute, parent robotiq_85_base_link, child robotiq_85_left_knuckle_link, origin xyz=0.05490451627 0.03060114443 0.0 rpy=3.141592653 0.0 0.0, axis 0 0 1, limit lower=-0.05 upper=0.80285 effort=1000 velocity=0.5
- added joint robotiq_85_right_finger_joint: type fixed, parent robotiq_85_right_knuckle_link, child robotiq_85_right_finger_link, origin xyz=-0.00408552455 -0.03148604435 0.0 rpy=0 0 0
- added joint robotiq_85_right_finger_tip_joint: type continuous, parent robotiq_85_right_inner_knuckle_link, child robotiq_85_right_finger_tip_link, origin xyz=0.04303959807 -0.03759940821  0.0 rpy=0.0 0.0 0.0, axis 0 0 1, limit lower=-0.80285 upper=0.05 effort=1000 velocity=0.5
- added joint robotiq_85_right_inner_knuckle_joint: type continuous, parent robotiq_85_base_link, child robotiq_85_right_inner_knuckle_link, origin xyz=0.06142 -0.0127 0 rpy=0 0 0, axis 0 0 1, limit lower=-0.05 upper=0.80285 effort=1000 velocity=0.5
- added joint robotiq_85_right_knuckle_joint: type continuous, parent robotiq_85_base_link, child robotiq_85_right_knuckle_link, origin xyz=0.05490451627 -0.03060114443 0.0 rpy=0.0 0.0 0.0, axis 0 0 1, limit lower=-0.05 upper=0.80285 effort=1000 velocity=0.5
- added joint robotiq_coupler_joint: type fixed, parent tool0, child robotiq_coupler, origin xyz=0 0 0.004 rpy=0 0 -1.57079632679

Commit message: minor

File: Universal_Robots/ur10_robotiq_2f_85/ur10_gripper.urdf (robot description, URDF)
Before this commit: robot ur10, 22 links, 21 joints
Links:
- link wrist_2_link: geometry collision mesh filename=./meshes/meshes/ur10/collision/wrist2.stl; visual mesh filename=./meshes/ur10/visual/wrist2.dae
- link wrist_3_link: geometry collision mesh filename=./meshes/ur10/collision/wrist3.stl; visual mesh filename=./meshes/ur10/visual/wrist3.dae

Commit message: minor

File: Universal_Robots/ur10_robotiq_2f_85/ur10_gripper.urdf (robot description, URDF)
Before this commit: robot ur10, 22 links, 21 joints
Links:
- link wrist_1_link: geometry collision mesh filename=./meshes/collision/Wrist1.dae; visual mesh filename=./meshes/visual/Wrist1.dae
- link wrist_2_link: geometry collision mesh filename=./meshes/collision/Wrist2.dae; visual mesh filename=./meshes/visual/Wrist2.dae
- link wrist_3_link: geometry collision mesh filename=./meshes/collision/Wrist3.dae; visual mesh filename=./meshes/visual/Wrist3.dae
Joints:
- joint robotiq_85_left_inner_knuckle_joint: origin xyz=0.06142 0.0127 0 rpy=${pi} 0.0 0.0 -> xyz=0.06142 0.0127 0 rpy=3.141592654 0.0 0.0

Commit message: minor

File: Universal_Robots/ur10_robotiq_2f_85/ur10_gripper.urdf (robot description, URDF)
Before this commit: robot ur10, 22 links, 21 joints
Links:
- link robotiq_85_base_link: geometry collision mesh filename=./meshes/robotiq2f85/robotiq_85_base_link_coarse.STL; visual mesh filename=./meshes/robotiq2f85/robotiq_85_base_link_fine.STL
- link robotiq_85_left_knuckle_link: geometry collision mesh filename=./meshes/robotiq2f85/outer_knuckle_coarse.stl; visual mesh filename=./meshes/robotiq2f85/outer_knuckle_coarse.stl
