Commit message: updated coke object

File: objects/coke.urdf (robot description, URDF)
Before this commit: robot coke, 1 links, 0 joints
Links:
- link body: geometry collision mesh filename=./meshes/coke.obj scale=1 1 0.8; visual mesh filename=./meshes/coke.obj scale=1 1 0.8

Commit message: minor

File: objects/coke.urdf (robot description, URDF)
Before this commit: robot coke, 1 links, 0 joints
Links:
- link body: geometry collision mesh filename=./meshes/coke.dae scale=1 1 0.8; visual mesh filename=./meshes/coke.dae scale=1 1 0.8
