Commit message: minor

File: objects/water_jar.urdf (robot description, URDF)
Before this commit: robot water_jar, 1 links, 0 joints
Links:
- link body: geometry collision mesh filename=meshes/water_jar.dae scale=0.6 0.6 1; visual mesh filename=meshes/water_jar.dae scale=0.6 0.6 1

Commit message: minor

File: objects/water_jar.urdf (robot description, URDF)
Before this commit: robot water_jar, 1 links, 0 joints
Links:
- link body: geometry collision mesh filename=./meshes/water_jar.obj scale=0.6 0.6 1; visual mesh filename=./meshes/water_jar.obj scale=0.6 0.6 1
