Commit message: minor

File: objects/waterjar.urdf (robot description, URDF)
Before this commit: robot water_jar, 1 links, 0 joints
Links:
- link body: geometry collision mesh filename=./meshes/waterjar.obj scale=0.6 0.6 1; visual mesh filename=./meshes/waterjar.obj scale=0.6 0.6 1

Commit message: minor

File: objects/waterjar.urdf (robot description, URDF)
Before this commit: robot water_jar, 1 links, 0 joints
Links:
- link body: mass 0.255 -> 0.050

Commit message: minor

File: objects/waterjar.urdf (robot description, URDF)
Before this commit: robot waterjar, 1 links, 0 joints
Links:
- link body: geometry collision mesh filename=./meshes/waterjar.obj scale=1 1 1; visual mesh filename=./meshes/waterjar.obj scale=1 1 1

Commit message: minor

File: objects/waterjar.urdf (robot description, URDF)
Before this commit: robot waterjar, 1 links, 0 joints
Links:
- link body: geometry collision mesh filename=./meshes/waterjar.obj scale=0.6 0.6 1.11; visual mesh filename=./meshes/waterjar.obj scale=0.6 0.6 1.11
